Commit message: pref: 分别添加了用于 IK 和全身预览的 urdf 和 meshes

File: urdf/lanchong_description.urdf (robot description, URDF)
Before this commit: robot lanchong_description, 28 links, 27 joints
Links:
- removed link front_left_roller_link
- removed link front_left_rudder_link
- removed link front_right_roller_link
- removed link front_right_rudder_link
- removed link left_clamp_left_link
- removed link left_clamp_right_link
- removed link neck_pitch_link
- removed link neck_yaw_link
- removed link pelvis_link
- removed link rear_middle_roller_link
- removed link rear_middle_rudder_link
- removed link right_clamp_left_link
- removed link right_clamp_right_link
- removed link vehicle
- added link pelvis, mass 8.8996; collision mesh filename=package://lanchong_description/meshes/pelvis.STL; visual mesh filename=package://lanchong_description/meshes/pelvis.STL
- link left_wrist_yaw_link: mass 0.18746 -> 0.25686
- link right_wrist_yaw_link: mass 0.18746 -> 0.25686
Joints:
- removed joint front_left_roller_joint
- removed joint front_left_rudder_joint
- removed joint front_right_roller_joint
- removed joint front_right_rudder_joint
- removed joint left_clamp_left_joint
- removed joint left_clamp_right_joint
- removed joint neck_pitch_joint
- removed joint neck_yaw_joint
- removed joint pelvis_joint
- removed joint rear_middle_roller_joint
- removed joint rear_middle_rudder_joint
- removed joint right_clamp_left_joint
- removed joint right_clamp_right_joint
- joint left_elbow_joint: limit lower=-2.477 upper=0.662 effort=100 velocity=1 -> lower=-3.14 upper=3.14 effort=100 velocity=1
- joint left_shoulder_pitch_joint: origin xyz=0 0.11533 0 rpy=0.43633 0 0 -> xyz=0 0.11533 0.78881 rpy=0.43633 0 0; parent pelvis_link -> pelvis
- joint left_wrist_pitch_joint: axis 0 0 1 -> 0 1 0; limit lower=-2.094 upper=2.094 effort=100 velocity=1 -> lower=-3.14 upper=3.14 effort=100 velocity=1
- joint left_wrist_yaw_joint: axis 0 1 0 -> 0 0 1; limit lower=-1.744 upper=1.744 effort=100 velocity=1 -> lower=-3.14 upper=3.14 effort=100 velocity=1
- joint right_elbow_joint: limit lower=-2.477 upper=0.662 effort=100 velocity=1 -> lower=-3.14 upper=3.14 effort=100 velocity=1
- joint right_shoulder_pitch_joint: origin xyz=0 -0.11533 0 rpy=-0.43633 0 0 -> xyz=0 -0.11533 0.78881 rpy=-0.43633 0 0; parent pelvis_link -> pelvis
- joint right_wrist_pitch_joint: axis 0 0 1 -> 0 1 0; limit lower=-2.094 upper=2.094 effort=100 velocity=1 -> lower=-3.14 upper=3.14 effort=100 velocity=1
- joint right_wrist_yaw_joint: axis 0 1 0 -> 0 0 1; limit lower=-1.744 upper=1.744 effort=100 velocity=1 -> lower=-3.14 upper=3.14 effort=100 velocity=1
