Commit message: chore(urdf): 删除自动生成的 mantis1.xacro 文件
该文件由 SolidWorks 导出工具自动生成，注释已说明不应手动编辑。
删除此文件以清理代码库，避免与手动维护的 URDF 文件产生混淆。

File: urdf/mantis.xacro (robot description, xacro)
@@ -1,47 +1,34 @@
-<?xml version="1.0" ?>
-<!-- =================================================================================== -->
-<!-- |    This document was autogenerated by xacro from $(find mantis_description).urdf                    | -->
-<!-- |    EDITING THIS FILE BY HAND IS NOT RECOMMENDED                                 | -->
-<!-- =================================================================================== -->
-<!-- This URDF was automatically created by SolidWorks to URDF Exporter! Originally created by Stephen Brawner (brawner@gmail.com)
-     Commit Version: 1.6.0-4-g7f85cfe  Build Version: 1.6.7995.38578
-     For more information, please see http://wiki.ros.org/sw_urdf_exporter -->
-<robot name="mantis">
-  <link name="world"/>
-  <joint name="world_to_base_footprint_joint" type="fixed">
-    <origin rpy="0 0 0" xyz="0 0 0"/>
-    <parent link="world"/>
-    <child link="base_footprint"/>
-  </joint>
+<?xml version="1.0" encoding="utf-8"?>
+<robot name="mantis" xmlns:xacro="http://www.ros.org/wiki/xacro">
   <link name="base_footprint">
     <inertial>
-      <mass value="0.001"/>
-      <inertia ixx="0.001" ixy="0.0" ixz="0.0" iyy="0.001" iyz="0.0" izz="0.001"/>
+      <mass value="0.001" />
+      <inertia ixx="0.001" ixy="0.0" ixz="0.0" iyy="0.001" iyz="0.0" izz="0.001" />
     </inertial>
   </link>
   <joint name="base_footprint_joint" type="fixed">
-    <origin rpy="0 0 0" xyz="0 0 1.01118"/>
-    <parent link="base_footprint"/>
-    <child link="base_link"/>
+    <origin xyz="0 0 0.91118" rpy="0 0 0" />
+    <parent link="base_footprint" />
+    <child link="base_link" />
   </joint>
   <link name="base_link">
     <inertial>
-      <origin rpy="0 0 0" xyz="0.00291835016733648 0.0443306772002185 -0.506676490095276"/>
-      <mass value="18.7682865290739"/>
-      <inertia ixx="1.01453122275419" ixy="-0.001292193416061" ixz="-0.00132472052415733" iyy="1.05820709577485" iyz="-0.00312229073177444" izz="0.14917498215046"/>
-    </inertial>
-    <visual>
-      <origin rpy="0 0 0" xyz="0 0 0"/>
-      <geometry>
-        <mesh filename="$(find mantis_description)/meshes/visual/base_link.STL"/>
-      </geometry>
-      <material name="">
-        <color rgba="0.792156862745098 0.819607843137255 0.933333333333333 1"/>
-      </material>
-    </visual>
-    <collision>
-      <origin rpy="0 0 0" xyz="0 0 0"/>
-      <geometry>
-        <mesh filename="$(find mantis_description)/meshes/visual/base_link.STL"/>
+      <origin xyz="0.00291835016733648 0.0443306772002185 -0.506676490095276" rpy="0 0 0" />
+      <mass value="18.7682865290739" />
+      <inertia ixx="1.01453122275419" ixy="-0.001292193416061" ixz="-0.00132472052415733" iyy="1.05820709577485" iyz="-0.00312229073177444" izz="0.14917498215046" />
+    </inertial>
+    <visual>
+      <origin xyz="0 0 0" rpy="0 0 0" />
+      <geometry>
+        <mesh filename="package://mantis_description/meshes/visual/base_link.STL" />
+      </geometry>
+      <material name="">
+        <color rgba="0.792156862745098 0.819607843137255 0.933333333333333 1" />
+      </material>
+    </visual>
+    <collision>
+      <origin xyz="0 0 0" rpy="0 0 0" />
+      <geometry>
+        <mesh filename="package://mantis_description/meshes/collision/base_link.STL" />
       </geometry>
     </collision>
@@ -49,834 +36,865 @@
   <link name="Waist_Link">
     <inertial>
-      <origin rpy="0 0 0" xyz="0.000667374250975017 0.0629984186385113 0.0843576330118845"/>
-      <mass value="1.99662648153202"/>
-      <inertia ixx="0.00509215547587237" ixy="-1.46364163321071E-06" ixz="3.01532372097028E-06" iyy="0.0094519829543267" iyz="-5.07590723983843E-05" izz="0.00610861474597361"/>
-    </inertial>
-    <visual>
-      <origin rpy="0 0 0" xyz="0 0 0"/>
-      <geometry>
-        <mesh filename="$(find mantis_description)/meshes/visual/Waist_Link.STL"/>
-      </geometry>
-      <material name="">
-        <color rgba="0.792156862745098 0.819607843137255 0.933333333333333 1"/>
-      </material>
-    </visual>
-    <collision>
-      <origin rpy="0 0 0" xyz="0 0 0"/>
-      <geometry>
-        <mesh filename="$(find mantis_description)/meshes/visual/Waist_Link.STL"/>
-      </geometry>
-    </collision>
-  </link>
-  <joint name="Waist_Joint" type="fixed">
-    <origin rpy="0 0 0" xyz="0 0 0"/>
-    <parent link="base_link"/>
-    <child link="Waist_Link"/>
-    <axis xyz="0 0 1"/>
-    <limit effort="100000" lower="-0.62" upper="0.24" velocity="100"/>
+      <origin xyz="0.000667374250975017 0.0629984186385113 0.0843576330118845" rpy="0 0 0" />
+      <mass value="1.99662648153202" />
+      <inertia ixx="0.00509215547587237" ixy="-1.46364163321071E-06" ixz="3.01532372097028E-06" iyy="0.0094519829543267" iyz="-5.07590723983843E-05" izz="0.00610861474597361" />
+    </inertial>
+    <visual>
+      <origin xyz="0 0 0" rpy="0 0 0" />
+      <geometry>
+        <mesh filename="package://mantis_description/meshes/visual/Waist_Link.STL" />
+      </geometry>
+      <material name="">
+        <color rgba="0.792156862745098 0.819607843137255 0.933333333333333 1" />
+      </material>
+    </visual>
+    <collision>
+      <origin xyz="0 0 0" rpy="0 0 0" />
+      <geometry>
+        <mesh filename="package://mantis_description/meshes/collision/Waist_Link.STL" />
+      </geometry>
+    </collision>
+  </link>
+  <joint name="Waist_Joint" type="prismatic">
+    <origin xyz="0 0 0" rpy="0 0 0" />
+    <parent link="base_link" />
+    <child link="Waist_Link" />
+    <axis xyz="0 0 1" />
+    <limit lower="-0.62" upper="0.24" effort="1000" velocity="10" />
   </joint>
   <link name="L_Shoulder_Pitch_Link">
     <inertial>
-      <origin rpy="0 0 0" xyz="0.0744985888480547 -0.00693271478878255 0.0731075230280795"/>
-      <mass value="0.372891915969362"/>
-      <inertia ixx="0.00106393418282301" ixy="-2.08105832368009E-06" ixz="-0.000267691987637077" iyy="0.00105100436144777" iyz="2.41936515367882E-05" izz="0.000785767690661667"/>
-    </inertial>
-    <visual>
-      <origin rpy="0 0 0" xyz="0 0 0"/>
-      <geometry>
-        <mesh filename="$(find mantis_description)/meshes/visual/L_Shoulder_Pitch_Link.STL"/>
-      </geometry>
-      <material name="">
-        <color rgba="0.792156862745098 0.819607843137255 0.933333333333333 1"/>
-      </material>
-    </visual>
-    <collision>
-      <origin rpy="0 0 0" xyz="0 0 0"/>
-      <geometry>
-        <mesh filename="$(find mantis_description)/meshes/visual/L_Shoulder_Pitch_Link.STL"/>
+      <origin xyz="0.0744985888480547 -0.00693271478878255 0.0731075230280795" rpy="0 0 0" />
+      <mass value="0.372891915969362" />
+      <inertia ixx="0.00106393418282301" ixy="-2.08105832368009E-06" ixz="-0.000267691987637077" iyy="0.00105100436144777" iyz="2.41936515367882E-05" izz="0.000785767690661667" />
+    </inertial>
+    <visual>
+      <origin xyz="0 0 0" rpy="0 0 0" />
+      <geometry>
+        <mesh filename="package://mantis_description/meshes/visual/L_Shoulder_Pitch_Link.STL" />
+      </geometry>
+      <material name="">
+        <color rgba="0.792156862745098 0.819607843137255 0.933333333333333 1" />
+      </material>
+    </visual>
+    <collision>
+      <origin xyz="0 0 0" rpy="0 0 0" />
+      <geometry>
+        <mesh filename="package://mantis_description/meshes/collision/L_Shoulder_Pitch_Link.STL" />
       </geometry>
     </collision>
   </link>
   <joint name="L_Shoulder_Pitch_Joint" type="revolute">
-    <origin rpy="1.13276835695949 -0.0851167590398302 -1.53099902329074" xyz="-0.119380687883944 0.112951840620579 0.138494616384493"/>
-    <parent link="Waist_Link"/>
-    <child link="L_Shoulder_Pitch_Link"/>
-    <axis xyz="0 0 -1"/>
-    <limit effort="100000" lower="-2.61" upper="0.78" velocity="100"/>
+    <origin xyz="-0.119380687883944 0.112951840620579 0.138494616384493" rpy="1.13276835695949 -0.0851167590398302 -1.53099902329074" />
+    <parent link="Waist_Link" />
+    <child link="L_Shoulder_Pitch_Link" />
+    <axis xyz="0 0 -1" />
+    <limit lower="-1.13" upper="1.75" effort="1000" velocity="10" />
   </joint>
   <link name="L_Shoulder_Yaw_Link">
     <inertial>
-      <origin rpy="0 0 0" xyz="0.000893474453819182 0.0235983806613933 0.0891963130495212"/>
-      <mass value="0.393421362351111"/>
-      <inertia ixx="0.000690227949322727" ixy="4.49819259821545E-07" ixz="-3.79368492386007E-07" iyy="0.0010958277239914" iyz="6.6243644536686E-06" izz="0.000511821421351544"/>
-    </inertial>
-    <visual>
-      <origin rpy="0 0 0" xyz="0 0 0"/>
-      <geometry>
-        <mesh filename="$(find mantis_description)/meshes/visual/L_Shoulder_Yaw_Link.STL"/>
-      </geometry>
-      <material name="">
-        <color rgba="0.792156862745098 0.819607843137255 0.933333333333333 1"/>
-      </material>
-    </visual>
-    <collision>
-      <origin rpy="0 0 0" xyz="0 0 0"/>
-      <geometry>
-        <mesh filename="$(find mantis_description)/meshes/visual/L_Shoulder_Yaw_Link.STL"/>
+      <origin xyz="0.000893474453819182 0.0235983806613933 0.0891963130495212" rpy="0 0 0" />
+      <mass value="0.393421362351111" />
+      <inertia ixx="0.000690227949322727" ixy="4.49819259821545E-07" ixz="-3.79368492386007E-07" iyy="0.0010958277239914" iyz="6.6243644536686E-06" izz="0.000511821421351544" />
+    </inertial>
+    <visual>
+      <origin xyz="0 0 0" rpy="0 0 0" />
+      <geometry>
+        <mesh filename="package://mantis_description/meshes/visual/L_Shoulder_Yaw_Link.STL" />
+      </geometry>
+      <material name="">
+        <color rgba="0.792156862745098 0.819607843137255 0.933333333333333 1" />
+      </material>
+    </visual>
+    <collision>
+      <origin xyz="0 0 0" rpy="0 0 0" />
+      <geometry>
+        <mesh filename="package://mantis_description/meshes/collision/L_Shoulder_Yaw_Link.STL" />
       </geometry>
     </collision>
   </link>
   <joint name="L_Shoulder_Yaw_Joint" type="revolute">
-    <origin rpy="1.57079632679492 -1.13446331231414 -1.66473705767284" xyz="0.0851253117883655 -0.00746534000720467 0.110000000000001"/>
-    <parent link="L_Shoulder_Pitch_Link"/>
-    <child link="L_Shoulder_Yaw_Link"/>
-    <axis xyz="0.00232272052559061 -0.00498108111894372 0.99998489678607"/>
-    <limit effort="100000" lower="0.08" upper="1.04" velocity="100"/>
+    <origin xyz="0.0851253117883655 -0.00746534000720467 0.110000000000001" rpy="1.57079632679492 -1.13446331231414 -1.66473705767284" />
+    <parent link="L_Shoulder_Pitch_Link" />
+    <child link="L_Shoulder_Yaw_Link" />
+    <axis xyz="0.00232272052559061 -0.00498108111894372 0.99998489678607" />
+    <limit lower="-0.213" upper="2.029" effort="1000" velocity="10" />
   </joint>
   <link name="L_Shoulder_Roll_Link">
     <inertial>
-      <origin rpy="0 0 0" xyz="0.000273423588430743 0.014504264229619 -0.156867248473735"/>
-      <mass value="0.695321962010077"/>
-      <inertia ixx="0.00222515527596948" ixy="-7.72037242091645E-06" ixz="-0.000237752894573366" iyy="0.00304543533311495" iyz="4.26548780737523E-07" izz="0.00097088400056944"/>
-    </inertial>
-    <visual>
-      <origin rpy="0 0 0" xyz="0 0 0"/>
-      <geometry>
-        <mesh filename="$(find mantis_description)/meshes/visual/L_Shoulder_Roll_Link.STL"/>
-      </geometry>
-      <material name="">
-        <color rgba="0.792156862745098 0.819607843137255 0.933333333333333 1"/>
-      </material>
-    </visual>
-    <collision>
-      <origin rpy="0 0 0" xyz="0 0 0"/>
-      <geometry>
-        <mesh filename="$(find mantis_description)/meshes/visual/L_Shoulder_Roll_Link.STL"/>
+      <origin xyz="0.000273423588430743 0.014504264229619 -0.156867248473735" rpy="0 0 0" />
+      <mass value="0.695321962010077" />
+      <inertia ixx="0.00222515527596948" ixy="-7.72037242091645E-06" ixz="-0.000237752894573366" iyy="0.00304543533311495" iyz="4.26548780737523E-07" izz="0.00097088400056944" />
+    </inertial>
+    <visual>
+      <origin xyz="0 0 0" rpy="0 0 0" />
+      <geometry>
+        <mesh filename="package://mantis_description/meshes/visual/L_Shoulder_Roll_Link.STL" />
+      </geometry>
+      <material name="">
+        <color rgba="0.792156862745098 0.819607843137255 0.933333333333333 1" />
+      </material>
+    </visual>
+    <collision>
+      <origin xyz="0 0 0" rpy="0 0 0" />
+      <geometry>
+        <mesh filename="package://mantis_description/meshes/collision/L_Shoulder_Roll_Link.STL" />
       </geometry>
     </collision>
   </link>
   <joint name="L_Shoulder_Roll_Joint" type="revolute">
-    <origin rpy="-1.46410662647607 -1.52400299359648 -0.106578883100582" xyz="0.000245013973831892 -0.00702542342111112 0.105466029573021"/>
-    <parent link="L_Shoulder_Yaw_Link"/>
-    <child link="L_Shoulder_Roll_Link"/>
-    <axis xyz="0 0 -1"/>
-    <limit effort="100000" lower="-1.57" upper="1.57" velocity="100"/>
+    <origin xyz="0.000245013973831892 -0.00702542342111112 0.105466029573021" rpy="-1.46410662647607 -1.52400299359648 -0.106578883100582" />
+    <parent link="L_Shoulder_Yaw_Link" />
+    <child link="L_Shoulder_Roll_Link" />
+    <axis xyz="0 0 -1" />
+    <limit lower="-0.8" upper="0.82" effort="1000" velocity="10" />
   </joint>
   <link name="L_Elbow_Pitch_Link">
     <inertial>
-      <origin rpy="0 0 0" xyz="-0.073954781690543 -0.0163741200998277 0.014115195798584"/>
-      <mass value="0.16496719809056"/>
-      <inertia ixx="8.93436041504421E-05" ixy="5.65092772192201E-06" ixz="3.27764279818126E-09" iyy="0.000107444526172469" iyz="2.66186893468467E-08" izz="0.000131201935224251"/>
-    </inertial>
-    <visual>
-      <origin rpy="0 0 0" xyz="0 0 0"/>
-      <geometry>
-        <mesh filename="$(find mantis_description)/meshes/visual/L_Elbow_Pitch_Link.STL"/>
-      </geometry>
-      <material name="">
-        <color rgba="0.792156862745098 0.819607843137255 0.933333333333333 1"/>
-      </material>
-    </visual>
-    <collision>
-      <origin rpy="0 0 0" xyz="0 0 0"/>
-      <geometry>
-        <mesh filename="$(find mantis_description)/meshes/visual/L_Elbow_Pitch_Link.STL"/>
+      <origin xyz="-0.073954781690543 -0.0163741200998277 0.014115195798584" rpy="0 0 0" />
+      <mass value="0.16496719809056" />
+      <inertia ixx="8.93436041504421E-05" ixy="5.65092772192201E-06" ixz="3.27764279818126E-09" iyy="0.000107444526172469" iyz="2.66186893468467E-08" izz="0.000131201935224251" />
+    </inertial>
+    <visual>
+      <origin xyz="0 0 0" rpy="0 0 0" />
+      <geometry>
+        <mesh filename="package://mantis_description/meshes/visual/L_Elbow_Pitch_Link.STL" />
+      </geometry>
+      <material name="">
+        <color rgba="0.792156862745098 0.819607843137255 0.933333333333333 1" />
+      </material>
+    </visual>
+    <collision>
+      <origin xyz="0 0 0" rpy="0 0 0" />
+      <geometry>
+        <mesh filename="package://mantis_description/meshes/collision/L_Elbow_Pitch_Link.STL" />
       </geometry>
     </collision>
   </link>
   <joint name="L_Elbow_Pitch_Joint" type="revolute">
-    <origin rpy="1.5707963267949 0.147258361384734 3.14159265358979" xyz="0 -0.0139999999999995 -0.35448"/>
-    <parent link="L_Shoulder_Roll_Link"/>
-    <child link="L_Elbow_Pitch_Link"/>
-    <axis xyz="0 0 1"/>
-    <limit effort="100000" lower="-0.78" upper="1.57" velocity="100"/>
+    <origin xyz="0 -0.0139999999999995 -0.35448" rpy="1.5707963267949 0.147258361384734 3.14159265358979" />
+    <parent link="L_Shoulder_Roll_Link" />
+    <child link="L_Elbow_Pitch_Link" />
+    <axis xyz="0 0 1" />
+    <limit lower="-0.395" upper="1.012" effort="1000" velocity="10" />
   </joint>
   <link name="L_Wrist_Roll_Link">
     <inertial>
-      <origin rpy="0 0 0" xyz="0.00727590094110392 -1.65127836166956E-05 0.0569761656185965"/>
-      <mass value="0.169478942795133"/>
-      <inertia ixx="0.000239103036527986" ixy="1.03758336805756E-07" ixz="-6.28682254541951E-06" iyy="0.000206064539212636" iyz="-3.42381105143778E-07" izz="8.205196326405E-05"/>
-    </inertial>
-    <visual>
-      <origin rpy="0 0 0" xyz="0 0 0"/>
-      <geometry>
-        <mesh filename="$(find mantis_description)/meshes/visual/L_Wrist_Roll_Link.STL"/>
-      </geometry>
-      <material name="">
-        <color rgba="0.792156862745098 0.819607843137255 0.933333333333333 1"/>
-      </material>
-    </visual>
-    <collision>
-      <origin rpy="0 0 0" xyz="0 0 0"/>
-      <geometry>
-        <mesh filename="$(find mantis_description)/meshes/visual/L_Wrist_Roll_Link.STL"/>
+      <origin xyz="0.00727590094110392 -1.65127836166956E-05 0.0569761656185965" rpy="0 0 0" />
+      <mass value="0.169478942795133" />
+      <inertia ixx="0.000239103036527986" ixy="1.03758336805756E-07" ixz="-6.28682254541951E-06" iyy="0.000206064539212636" iyz="-3.42381105143778E-07" izz="8.205196326405E-05" />
+    </inertial>
+    <visual>
+      <origin xyz="0 0 0" rpy="0 0 0" />
+      <geometry>
+        <mesh filename="package://mantis_description/meshes/visual/L_Wrist_Roll_Link.STL" />
+      </geometry>
+      <material name="">
+        <color rgba="0.792156862745098 0.819607843137255 0.933333333333333 1" />
+      </material>
+    </visual>
+    <collision>
+      <origin xyz="0 0 0" rpy="0 0 0" />
+      <geometry>
+        <mesh filename="package://mantis_description/meshes/collision/L_Wrist_Roll_Link.STL" />
       </geometry>
     </collision>
   </link>
   <joint name="L_Wrist_Roll_Joint" type="revolute">
-    <origin rpy="1.27728583452051 -1.57079630572147 -1.09751485724235" xyz="-0.127614538662876 -0.0220177037533985 0.0139999999999991"/>
-    <parent link="L_Elbow_Pitch_Link"/>
-    <child link="L_Wrist_Roll_Link"/>
-    <axis xyz="0 0 1"/>
-    <limit effort="100000" lower="-1.57" upper="1.57" velocity="100"/>
+    <origin xyz="-0.127614538662876 -0.0220177037533985 0.0139999999999991" rpy="1.27728583452051 -1.57079630572147 -1.09751485724235" />
+    <parent link="L_Elbow_Pitch_Link" />
+    <child link="L_Wrist_Roll_Link" />
+    <axis xyz="0 0 1" />
+    <limit lower="-1.7" upper="1.7" effort="1000" velocity="10" />
   </joint>
   <link name="L_Wrist_Pitch_Link">
     <inertial>
-      <origin rpy="0 0 0" xyz="0.000108166573202562 0.00197671902424157 0.0335770575398197"/>
-      <mass value="0.0628660572692061"/>
-      <inertia ixx="1.93938974724344E-05" ixy="4.66755021966573E-08" ixz="2.43928519334516E-07" iyy="2.82007568195928E-05" iyz="-8.08379103988105E-08" izz="1.82253216552244E-05"/>
-    </inertial>
-    <visual>
-      <origin rpy="0 0 0" xyz="0 0 0"/>
-      <geometry>
-        <mesh filename="$(find mantis_description)/meshes/visual/L_Wrist_Pitch_Link.STL"/>
-      </geometry>
-      <material name="">
-        <color rgba="0.792156862745098 0.819607843137255 0.933333333333333 1"/>
-      </material>
-    </visual>
-    <collision>
-      <origin rpy="0 0 0" xyz="0 0 0"/>
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